File: CAD/電路LAYOUT/24_TDK_Syno/Syno_Ver1.0.brd (EAGLE design)
At the start: 55.9 x 65.7 mm, 13 parts, among them IC1 REG1117

Commit message: daily update
整理檔案與更新電路Layout(1.0~1.2)
Parts:
- moved PWM_OUTPUT 1.27 mm to (10.2, 0.00)
Routing:
- net N$7: track 61.4 -> 67.1 mm
- net N$9: track 21.3 -> 26.4 mm
- net N$8: track 18.3 -> 21.1 mm
- net 5V_S: track 96.7 -> 98.3 mm
- net N$10: track 16.0 -> 17.3 mm
- net N$13: track 8.67 -> 9.94 mm
- net N$11: track 15.9 -> 16.4 mm
- net N$12: track 15.9 -> 16.4 mm
- removed copper zone on layer 1, net ASD
