File: CAD/電路LAYOUT/24_TDK_Syno/Syno_Ver1.2.sch (EAGLE design)
At the start: 13 parts, among them IC1 REG1117, X1 JST-XH-08-PIN-ROUND-PAD

Commit message: daily update
整理檔案與更新電路Layout(1.0~1.2)
Parts:
- removed JP1: (no value), pinhead:PINHD-1X7/90
- removed JP2: (no value), pinhead:PINHD-1X6/90
- removed X1: JST-XH-08-PIN-ROUND-PAD, Rembrandt Electronics - JST XH Connectors v1-0:JST-XH-08-PIN-ROUND-PAD
- added PIN: nRF24L01, Rembrandt Electronics - JST XH Connectors v1-0:JST-XH-08-PIN-ROUND-PAD
- added PWM_OUTPUT, RC_INPUT: (no value), pinhead:PINHD-1X7/90
- C1, C2: value (none) -> 10
Connections:
- new net N$1: MEGA2560PRO1.D51, PIN-3.S
- new net N$10: MEGA2560PRO1.D7, PWM_OUTPUT.4
- new net N$11: MEGA2560PRO1.D5, PWM_OUTPUT.5
- new net N$12: MEGA2560PRO1.D3, PWM_OUTPUT.6
- new net N$13: MEGA2560PRO1.A9, RC_INPUT.3
- new net N$14: MEGA2560PRO1.A7, RC_INPUT.4
- new net N$15: MEGA2560PRO1.A5, RC_INPUT.5
- new net N$16: MEGA2560PRO1.A3, RC_INPUT.6
- new net N$17: MEGA2560PRO1.A1, RC_INPUT.7
- new net N$2: C2.+, IC1.VOUT, PIN-1.S
- new net N$3: MEGA2560PRO1.D50, PIN-4.S
- new net N$4: MEGA2560PRO1.D52, PIN-5.S
- new net N$5: MEGA2560PRO1.D47, PIN-6.S
- new net N$6: MEGA2560PRO1.D46, PIN-7.S
- new net N$7: MEGA2560PRO1.D13, PWM_OUTPUT.1
- new net N$8: MEGA2560PRO1.D11, PWM_OUTPUT.2
- new net N$9: MEGA2560PRO1.D9, PWM_OUTPUT.3
- net 5V: now also MEGA2560PRO1.5V@1, MEGA2560PRO1.5V@2, RC_INPUT.1
- net 5V_S: now also C1.+, IC1.VIN
- net GND: now also MEGA2560PRO1.GND@1, MEGA2560PRO1.GND@2, PWM_OUTPUT.7, RC_INPUT.2
- net GND_S: now also C1.-, C2.-, IC1.GND, PIN-2.S
Other:
- moved on the sheet: C1, C2, IC1, POWER_MC
