File: CAD/電路LAYOUT/24_TDK_Syno/Syno_Ver2.0.brd (EAGLE design)
At the start: 63.2 x 54.6 mm, 17 parts, among them IC1 REG1117

Commit message: daily update
daily update
Parts:
- moved PWM_OUTPUT 1.27 mm to (29.2, 0.00)
- moved RC_INPUT 1.27 mm to (48.3, 0.00)
Routing:
- net N$15: track 5.39 -> 6.66 mm
- net N$16: track 5.39 -> 6.66 mm
- net N$17: track 5.39 -> 6.66 mm
- net N$14: track 5.39 -> 6.66 mm
- net N$18: track 5.39 -> 6.66 mm
- net N$19: track 5.39 -> 6.66 mm
- net MC_GND: track 51.5 -> 52.8 mm
- net MC_5V: track 87.8 -> 89.1 mm
- net N$24: track 3.81 -> 4.34 mm
- net N$23: track 3.81 -> 4.34 mm
- net N$22: track 3.81 -> 4.34 mm
- net N$21: track 3.81 -> 4.34 mm
- net N$20: track 3.81 -> 4.34 mm
Changed lines of the file:
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@@
 <attribute name="VALUE" x="43.815" y="48.26" size="1.27" layer="27" rot="R90"/>
 </element>
-<element name="PWM_OUTPUT" library="pinhead" library_urn="urn:adsk.eagle:library:325" package="1X07/90" package3d_urn="urn:adsk.eagle:package:22476/2" value="" x="27.94" y="0" smashed="yes" rot="R180">
-<attribute name="NAME" x="35.56" y="-8.255" size="1.27" layer="25" ratio="10" rot="R180"/>
-<attribute name="POPULARITY" value="1" x="-5.08" y="48.26" size="1.778" layer="27" rot="R180" display="off"/>
-<attribute name="VALUE" x="17.145" y="3.81" size="1.27" layer="27" rot="R270"/>
+<element name="PWM_OUTPUT" library="pinhead" library_urn="urn:adsk.eagle:library:325" package="1X07/90" package3d_urn="urn:adsk.eagle:package:22476/2" value="" x="29.21" y="0" smashed="yes" rot="R180">
+<attribute name="NAME" x="36.83" y="-8.255" size="1.27" layer="25" ratio="10" rot="R180"/>
+<attribute name="POPULARITY" value="1" x="-3.81" y="48.26" size="1.778" layer="27" rot="R180" display="off"/>
+<attribute name="VALUE" x="18.415" y="3.81" size="1.27" layer="27" rot="R270"/>
 </element>
 <element name="R1" library="rcl" library_urn="urn:adsk.eagle:library:334" package="0204/5" package3d_urn="urn:adsk.eagle:package:23488/1" value="20k" x="17.78" y="48.26" smashed="yes" rot="R270">
@@
 <attribute name="VALUE" x="25.05638125" y="51.9291375" size="0.9906" layer="27" ratio="10" rot="R225"/>
 </element>
-<element name="RC_INPUT" library="pinhead" library_urn="urn:adsk.eagle:library:325" package="1X07/90" package3d_urn="urn:adsk.eagle:package:22476/2" value="" x="46.99" y="0" smashed="yes" rot="R180">
-<attribute name="NAME" x="52.07" y="-8.255" size="1.27" layer="25" ratio="10" rot="R180"/>
-<attribute name="POPULARITY" value="1" x="-6.35" y="48.26" size="1.778" layer="27" rot="R180" display="off"/>
-<attribute name="VALUE" x="36.195" y="3.81" size="1.27" layer="27" rot="R270"/>
+<element name="RC_INPUT" library="pinhead" library_urn="urn:adsk.eagle:library:325" package="1X07/90" package3d_urn="urn:adsk.eagle:package:22476/2" value="" x="48.26" y="0" smashed="yes" rot="R180">
+<attribute name="NAME" x="53.34" y="-8.255" size="1.27" layer="25" ratio="10" rot="R180"/>
+<attribute name="POPULARITY" value="1" x="-5.08" y="48.26" size="1.778" layer="27" rot="R180" display="off"/>
+<attribute name="VALUE" x="37.465" y="3.81" size="1.27" layer="27" rot="R270"/>
 </element>
 <element name="SANDBAG_ACTUTOR" library="L9110" package="L9110H" value="L9110H" x="6.35" y="21.59" smashed="yes"/>
@@
 <wire x1="7.62" y1="3.81" x2="11.4505" y2="3.81" width="0.254" layer="1"/>
 <wire x1="11.4505" y1="3.81" x2="11.498" y2="3.7625" width="0.254" layer="1"/>
-<wire x1="57.15" y1="3.81" x2="57.15" y2="12.7" width="0.254" layer="1"/>
-<wire x1="57.15" y1="12.7" x2="11.43" y2="12.7" width="0.254" layer="1"/>
 <contactref element="MEGA2560PRO1" pad="5V@2"/>
+<wire x1="55.88" y1="12.7" x2="57.15" y2="12.7" width="0.254" layer="1"/>
+<wire x1="11.43" y1="12.7" x2="54.61" y2="12.7" width="0.254" layer="1"/>
+<wire x1="54.61" y1="12.7" x2="55.88" y2="12.7" width="0.254" layer="1"/>
 <wire x1="8.89" y1="10.16" x2="8.89" y2="7.62" width="0.254" layer="1"/>
 <wire x1="8.89" y1="10.16" x2="11.43" y2="12.7" width="0.254" layer="1"/>
 <contactref element="RC_INPUT" pad="6"/>
-<wire x1="41.91" y1="3.81" x2="41.91" y2="1.27" width="0.254" layer="1"/>
-<wire x1="41.91" y1="1.27" x2="54.61" y2="1.27" width="0.254" layer="1"/>
-<wire x1="54.61" y1="1.27" x2="57.15" y2="3.81" width="0.254" layer="1"/>
+<wire x1="43.18" y1="3.81" x2="43.18" y2="1.27" width="0.254" layer="1"/>
+<wire x1="43.18" y1="1.27" x2="57.15" y2="1.27" width="0.254" layer="1"/>
+<wire x1="58.42" y1="2.54" x2="57.15" y2="1.27" width="0.254" layer="1"/>
+<wire x1="57.15" y1="12.7" x2="58.42" y2="11.43" width="0.254" layer="1"/>
+<wire x1="58.42" y1="11.43" x2="58.42" y2="2.54" width="0.254" layer="1"/>
 </signal>
 <signal name="MC_GND">
@@
 <wire x1="2.54" y1="1.143" x2="13.843" y2="1.143" width="0.254" layer="1"/>
 <wire x1="13.498" y1="1.27" x2="13.97" y2="1.27" width="0.254" layer="1"/>
-<wire x1="13.97" y1="1.27" x2="20.32" y2="1.27" width="0.254" layer="1"/>
-<wire x1="20.32" y1="3.81" x2="20.32" y2="1.27" width="0.254" layer="1"/>
+<wire x1="13.97" y1="1.27" x2="21.59" y2="1.27" width="0.254" layer="1"/>
+<wire x1="21.59" y1="3.81" x2="21.59" y2="1.27" width="0.254" layer="1"/>
 <contactref element="RC_INPUT" pad="7"/>
-<wire x1="20.32" y1="1.27" x2="36.83" y2="1.27" width="0.254" layer="1"/>
-<wire x1="36.83" y1="1.27" x2="39.37" y2="3.81" width="0.254" layer="1"/>
+<wire x1="21.59" y1="1.27" x2="38.1" y2="1.27" width="0.254" layer="1"/>
+<wire x1="38.1" y1="1.27" x2="40.64" y2="3.81" width="0.254" layer="1"/>
 </signal>
 <signal name="N$11">
@@
 <contactref element="MEGA2560PRO1" pad="D3"/>
 <contactref element="PWM_OUTPUT" pad="6"/>
-<wire x1="19.05" y1="7.62" x2="22.86" y2="3.81" width="0.254" layer="1"/>
+<wire x1="24.13" y1="3.81" x2="21.59" y2="6.35" width="0.254" layer="1"/>
+<wire x1="21.59" y1="6.35" x2="20.32" y2="6.35" width="0.254" layer="1"/>
+<wire x1="19.05" y1="7.62" x2="20.32" y2="6.35" width="0.254" layer="1"/>
 </signal>
 <signal name="N$15">
 <contactref element="MEGA2560PRO1" pad="D5"/>
 <contactref element="PWM_OUTPUT" pad="5"/>
-<wire x1="21.59" y1="7.62" x2="25.4" y2="3.81" width="0.254" layer="1"/>
+<wire x1="26.67" y1="3.81" x2="24.13" y2="6.35" width="0.254" layer="1"/>
+<wire x1="24.13" y1="6.35" x2="22.86" y2="6.35" width="0.254" layer="1"/>
+<wire x1="21.59" y1="7.62" x2="22.86" y2="6.35" width="0.254" layer="1"/>
 </signal>
 <signal name="N$16">
 <contactref element="MEGA2560PRO1" pad="D7"/>
 <contactref element="PWM_OUTPUT" pad="4"/>
-<wire x1="24.13" y1="7.62" x2="27.94" y2="3.81" width="0.254" layer="1"/>
+<wire x1="29.21" y1="3.81" x2="26.67" y2="6.35" width="0.254" layer="1"/>
+<wire x1="26.67" y1="6.35" x2="25.4" y2="6.35" width="0.254" layer="1"/>
+<wire x1="24.13" y1="7.62" x2="25.4" y2="6.35" width="0.254" layer="1"/>
 </signal>
 <signal name="N$17">
 <contactref element="MEGA2560PRO1" pad="D9"/>
 <contactref element="PWM_OUTPUT" pad="3"/>
-<wire x1="26.67" y1="7.62" x2="30.48" y2="3.81" width="0.254" layer="1"/>
+<wire x1="31.75" y1="3.81" x2="29.21" y2="6.35" width="0.254" layer="1"/>
+<wire x1="29.21" y1="6.35" x2="27.94" y2="6.35" width="0.254" layer="1"/>
+<wire x1="26.67" y1="7.62" x2="27.94" y2="6.35" width="0.254" layer="1"/>
 </signal>
 <signal name="N$18">
 <contactref element="MEGA2560PRO1" pad="D11"/>
 <contactref element="PWM_OUTPUT" pad="2"/>
-<wire x1="29.21" y1="7.62" x2="33.02" y2="3.81" width="0.254" layer="1"/>
+<wire x1="34.29" y1="3.81" x2="31.75" y2="6.35" width="0.254" layer="1"/>
+<wire x1="31.75" y1="6.35" x2="30.48" y2="6.35" width="0.254" layer="1"/>
+<wire x1="29.21" y1="7.62" x2="30.48" y2="6.35" width="0.254" layer="1"/>
 </signal>
 <signal name="N$19">
 <contactref element="MEGA2560PRO1" pad="D13"/>
 <contactref element="PWM_OUTPUT" pad="1"/>
-<wire x1="31.75" y1="7.62" x2="35.56" y2="3.81" width="0.254" layer="1"/>
+<wire x1="36.83" y1="3.81" x2="34.29" y2="6.35" width="0.254" layer="1"/>
+<wire x1="31.75" y1="7.62" x2="33.02" y2="6.35" width="0.254" layer="1"/>
+<wire x1="34.29" y1="6.35" x2="33.02" y2="6.35" width="0.254" layer="1"/>
 </signal>
 <signal name="N$20">
 <contactref element="MEGA2560PRO1" pad="D23"/>
 <contactref element="RC_INPUT" pad="5"/>
-<wire x1="44.45" y1="7.62" x2="44.45" y2="3.81" width="0.254" layer="1"/>
+<wire x1="44.45" y1="7.62" x2="45.72" y2="6.35" width="0.254" layer="1"/>
+<wire x1="45.72" y1="6.35" x2="45.72" y2="3.81" width="0.254" layer="1"/>
 </signal>
 <signal name="N$21">
 <contactref element="MEGA2560PRO1" pad="D25"/>
 <contactref element="RC_INPUT" pad="4"/>
-<wire x1="46.99" y1="7.62" x2="46.99" y2="3.81" width="0.254" layer="1"/>
+<wire x1="46.99" y1="7.62" x2="48.26" y2="6.35" width="0.254" layer="1"/>
+<wire x1="48.26" y1="6.35" x2="48.26" y2="3.81" width="0.254" layer="1"/>
 </signal>
 <signal name="N$22">
 <contactref element="MEGA2560PRO1" pad="D27"/>
 <contactref element="RC_INPUT" pad="3"/>
-<wire x1="49.53" y1="7.62" x2="49.53" y2="3.81" width="0.254" layer="1"/>
+<wire x1="49.53" y1="7.62" x2="50.8" y2="6.35" width="0.254" layer="1"/>
+<wire x1="50.8" y1="6.35" x2="50.8" y2="3.81" width="0.254" layer="1"/>
 </signal>
 <signal name="N$23">
 <contactref element="MEGA2560PRO1" pad="D29"/>
 <contactref element="RC_INPUT" pad="2"/>
-<wire x1="52.07" y1="7.62" x2="52.07" y2="3.81" width="0.254" layer="1"/>
+<wire x1="52.07" y1="7.62" x2="53.34" y2="6.35" width="0.254" layer="1"/>
+<wire x1="53.34" y1="6.35" x2="53.34" y2="3.81" width="0.254" layer="1"/>
 </signal>
 <signal name="N$24">
 <contactref element="MEGA2560PRO1" pad="D31"/>
 <contactref element="RC_INPUT" pad="1"/>
-<wire x1="54.61" y1="7.62" x2="54.61" y2="3.81" width="0.254" layer="1"/>
+<wire x1="54.61" y1="7.62" x2="55.88" y2="6.35" width="0.254" layer="1"/>
+<wire x1="55.88" y1="6.35" x2="55.88" y2="3.81" width="0.254" layer="1"/>
 </signal>
 <signal name="N$25">
